File: PCBA/V2 Solenoid Engine PCB.kicad_sch (KiCad schematic)
At the start: 35 parts, among them J1 Screw_Terminal_01x02, J2 Screw_Terminal_01x02, J3 Screw_Terminal_01x02, J4 Screw_Terminal_01x02, J5 Solenoid B, J6 Solenoid A, J7 Screw_Terminal_01x02, Q1 IRFZ44N, Q2 IRFZ44N, U1 ESP32-DEVKIT-V1, U2 TC4427xOA, U5 TCRT5000, U6 TCRT5000

Commit message: Add files via upload
Connections:
- net GND: now also +24V_IN1.2 (Pin_2), C1.2, C2.2, C3.2, C4.2
- net at J6.1 (Pin_1): now also +24V_IN1.1 (Pin_1), CR1.2, CR2.2, F1.2, J5.1 (Pin_1)
- net at J6.2 (Pin_2): now also CR1.1
- net at CR2.1: now also J5.2 (Pin_2)
- net at C3.1: now also C1.1, C2.1, C4.1, F1.1
- no-connect marks 42 -> 21
